File: WLED-Salon/WLED-Salon.kicad_sch (KiCad schematic)
At the start: 2 parts, among them U1 ESP32-DevKitC, U2 74AHCT125

Commit message: schematic advancements
Parts:
- added C1, C2: 1000uF 16V, symbol Device:C_Polarized
- added C3: 100nF, symbol Device:C
- added F1, F2: Fuse 5A, symbol Device:Fuse
- added J1: 12V Power Supply, symbol Connector:Screw_Terminal_01x02
- added J2: Buck Converter, symbol Connector_Generic:Conn_01x04
- added J3: Power LED Strip 1, symbol Connector:Screw_Terminal_01x02
- added J4: Power LED Strip 2, symbol Connector:Screw_Terminal_01x02
- added J5: LED Strip Data 1 & 2, symbol Connector:Screw_Terminal_01x02
- added R1, R2: 62 Ohm, symbol Device:R_US
- added unit 4 of U2
- added U3: 74AHCT125, Package_DIP:DIP-14_W7.62mm_Socket, symbol 74xx:74AHCT125
Connections:
- net GND: now reaches U2.4
- net GND: now also U1.14 (GND), U1.32 (GND), U1.38 (GND), U2.1, U2.7 (GND), C1.2, C2.2, C3.2, J1.2 (Pin_2), J2.2 (Pin_2), J3.2 (Pin_2), J4.2 (Pin_2), U2.12, U3.9
- net GPIO17: now reaches U2.5
- net GPIO17: now also U1.28 (GPIO17)
- net at U2.6: now also R2.1
- net GPIO16: now reaches U2.2
- net GPIO16: now also U1.27 (GPIO16)
- net at U2.3: now also R1.1
- net +5V: now reaches U2.14 (VCC)
- net +5V: now also U1.19 (5V), C3.1, J2.1 (Pin_1), U2.13, U3.10
- new net: C2.1, F2.2, J4.1 (Pin_1)
- new net: C1.1, F1.2, J3.1 (Pin_1)
- new net +12V: F1.1, F2.1, J1.1 (Pin_1), J2.3 (Pin_3)
- new net DATA1: J5.1 (Pin_1), R1.2
- new net DATA2: J5.2 (Pin_2), R2.2
- no-connect marks 0 -> 35
Other:
- moved on the sheet: U1, U2A, U2B, U2E
